File: flipdot.kicad_pcb (KiCad board)
At the start: 2 copper layers, 16 parts, among them J5 Conn_01x04_Female, J6 Conn_01x02_Male, J7 Conn_01x02_Male, J8 Conn_02x30_Odd_Even, U1 WeMos_D1_mini

Commit message: update footprints
Parts:
- added J9: Conn_02x30_Odd_Even, Connector_PinHeader_2.54mm:PinHeader_2x30_P2.54mm_Vertical, F.Cu at (31.8, 25.4)
- added U8: FPF2702MX, Package_SO:SOIC-8_3.9x4.9mm_P1.27mm, F.Cu at (96.5, 86.4)
- J5: value Conn_01x04_Female -> Conn_01x02_Male; footprint Connector_PinHeader_2.54mm:PinHeader_1x04_P2.54mm_Vertical -> Connector_PinHeader_2.54mm:PinHeader_1x02_P2.54mm_Vertical
- J7: value Conn_01x02_Male -> Conn_02x30_Odd_Even; footprint Connector_PinHeader_2.54mm:PinHeader_1x02_P2.54mm_Vertical -> Connector_PinHeader_2.54mm:PinHeader_2x30_P2.54mm_Vertical
- J8: value Conn_02x30_Odd_Even -> Conn_01x04; footprint Connector_PinHeader_2.54mm:PinHeader_2x30_P2.54mm_Vertical -> Connector_PinHeader_2.54mm:PinHeader_1x04_P2.54mm_Vertical
- R3: value 10K -> 180
- R4: value 100K -> 150
- R5: value 10K -> 100K
- R6: value 180 -> 120
- R7: value 150 -> 10K
- R8: value 120 -> 10K
- U1: value WeMos_D1_mini -> 74HC595
- moved D2 338.3 mm to (85.6, 115.6)
- moved J7 335.8 mm to (31.8, 34.3), turned to 90 degrees
- moved D3 324.9 mm to (85.6, 113.0)
- moved R1 298.5 mm to (113.0, 114.3), turned to 180 degrees
- moved R6 295.1 mm to (82.1, 113.3)
- moved R4 290.7 mm to (82.1, 115.8)
- moved R3 289.4 mm to (82.1, 118.4)
- moved U1 281.6 mm to (108.0, 105.4)
- moved R7 276.0 mm to (92.7, 90.9)
- moved J8 260.7 mm to (109.2, 88.9), turned to 90 degrees
- moved R5 260.7 mm to (96.5, 81.3), turned to 180 degrees
- moved R2 259.8 mm to (90.2, 87.1), turned to 90 degrees
- moved J6 257.9 mm to (113.0, 30.5)
- moved R8 257.4 mm to (116.6, 114.3)
- moved J5 250.0 mm to (113.0, 22.9)
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Connections:
- J5 pad 1: Net-(J5-Pad1) -> 24V
- J5 pad 2: Net-(J5-Pad2) -> Net-(C1-Pad1)
- J6 pad 1: 24V -> Net-(C3-Pad1)
- J6 pad 2: Net-(C1-Pad1) -> VS
- J7 pad 1: VS -> SR1_ROW1_SET
- J7 pad 2: (no net) -> SR2_ROW2_SET
- R1 pad 1: 3V3 -> VCC
- R1 pad 2: EN_POWER_RAILS -> OE_5V
- R2 pad 1: (no net) -> Net-(R2-Pad1)
- R3 pad 1: VCC -> (no net)
- R3 pad 2: (no net) -> Net-(D1-Pad1)
- R4 pad 1: Net-(C1-Pad1) -> (no net)
- R4 pad 2: (no net) -> Net-(D2-Pad1)
- R5 pad 1: VCC -> Net-(R5-Pad1)
- R5 pad 2: (no net) -> Net-(C1-Pad1)
- R6 pad 2: Net-(D1-Pad1) -> Net-(D3-Pad1)
- R7 pad 2: Net-(D2-Pad1) -> EN_POWER_RAILS
- R8 pad 1: (no net) -> VCC
- R8 pad 2: Net-(D3-Pad1) -> (no net)
- U1 pad 1: Net-(U1-Pad1) -> (no net)
- U1 pad 10: GND -> (no net)
- U1 pad 11: Net-(J5-Pad2) -> (no net)
- U1 pad 13: (no net) -> OE_5V
- U1 pad 14: EN_POWER_RAILS -> (no net)
- U1 pad 15: Net-(J5-Pad3) -> (no net)
- U1 pad 16: Net-(J5-Pad4) -> VCC
- U1 pad 2: Net-(J5-Pad1) -> (no net)
- U1 pad 3: Net-(U1-Pad1) -> (no net)
- U1 pad 8: 3V3 -> GND
- U1 pad 9: VCC -> (no net)
Other:
- board outline added: 100 x 100 mm

Commit message: update
Parts:
- added C1: 100uF/35v, Capacitor_SMD:CP_Elec_6.3x7.7, F.Cu at (91.9, 109.7)
- added C2: 100u, Capacitor_THT:CP_Radial_D6.3mm_P2.50mm, F.Cu at (19.3, 68.6)
- added C3: 22u, Capacitor_THT:CP_Radial_D5.0mm_P2.00mm, F.Cu at (1.02, 59.4)
- added J1: 3V3, Connector_PinHeader_2.54mm:PinHeader_1x02_P2.54mm_Vertical, F.Cu at (70.1, 112.3)
- added J2: 5V, Connector_PinHeader_2.54mm:PinHeader_1x02_P2.54mm_Vertical, F.Cu at (74.2, 112.3)
- added J3: 24V, Connector_PinHeader_2.54mm:PinHeader_1x02_P2.54mm_Vertical, F.Cu at (78.2, 112.3)
- added J4: EN_PWR, Connector_PinHeader_2.54mm:PinHeader_1x02_P2.54mm_Vertical, F.Cu at (82.3, 112.3)
- added U10: ULN2803A, Package_SO:SOIC-18W_7.5x11.6mm_P1.27mm, F.Cu at (71.6, 43.2)
- added U11: ULN2803A, Package_SO:SOIC-18W_7.5x11.6mm_P1.27mm, F.Cu at (81.3, 57.4)
- added U12: A2982, Package_SO:SOIC-20W_7.5x12.8mm_P1.27mm, F.Cu at (65.5, 73.2)
- added U13: A2982, Package_SO:SOIC-20W_7.5x12.8mm_P1.27mm, F.Cu at (89.4, 43.2)
- added U14: A2982, Package_SO:SOIC-20W_7.5x12.8mm_P1.27mm, F.Cu at (102.1, 43.2)
- added U15: WeMos_D1_mini, wemos:wemos-d1-mini-with-pin-header-and-connector, F.Cu at (31.5, 101.1)
- added U16: ULN2803A, Package_SO:SOIC-18W_7.5x11.6mm_P1.27mm, F.Cu at (32.5, 44.7)
- added U17: ULN2803A, Package_SO:SOIC-18W_7.5x11.6mm_P1.27mm, F.Cu at (48.3, 44.7)
- added U18: 74HC245, Package_SO:SOP-20_7.5x12.8mm_P1.27mm, F.Cu at (33.5, 70.6)
- added U2: 74HC595, Package_SO:SOIC-16_3.9x9.9mm_P1.27mm, F.Cu at (93.0, 57.9)
- added U3: 74HC595, Package_SO:SOIC-16_3.9x9.9mm_P1.27mm, F.Cu at (47.2, 68.6)
- added U4: 74HC595, Package_SO:SOIC-16_3.9x9.9mm_P1.27mm, F.Cu at (73.2, 57.4)
- added U5: 74HC595, Package_SO:SOIC-16_3.9x9.9mm_P1.27mm, F.Cu at (58.9, 58.4)
- added U6: 74HC595, Package_SO:SOIC-16_3.9x9.9mm_P1.27mm, F.Cu at (46.7, 58.4)
- added U7: 74HC595, Package_SO:SOIC-16_3.9x9.9mm_P1.27mm, F.Cu at (32.0, 58.9)
- added U9: ULN2803A, Package_SO:SOIC-18W_7.5x11.6mm_P1.27mm, F.Cu at (61.5, 45.2)
- D1: value LED C RED -> LED C; footprint LED_SMD:LED_0603_1608Metric -> LED_SMD:LED_0805_2012Metric
- D2: value LED B YELLOW -> LED B; footprint LED_SMD:LED_0603_1608Metric -> LED_SMD:LED_0805_2012Metric
- D3: value LED A GREEN -> LED A; footprint LED_SMD:LED_0603_1608Metric -> LED_SMD:LED_0805_2012Metric
- R1, R7, R8: footprint Resistor_SMD:R_0603_1608Metric -> Resistor_SMD:R_0805_2012Metric
- R4: value 150 -> 180
- R6: value 120 -> 180
- U1: footprint wemos:wemos-d1-mini-with-pin-header-and-connector -> Package_SO:SOIC-16_3.9x9.9mm_P1.27mm
- moved J8 78.8 mm to (30.5, 85.3), turned to 270 degrees
- moved J7 73.5 mm to (105.2, 31.0), turned to 270 degrees
- moved J9 73.4 mm to (105.2, 23.9), turned to 270 degrees
- moved R8 68.0 mm to (56.3, 82.8)
- moved J6 67.3 mm to (107.2, 97.5)
- moved J5 66.3 mm to (107.2, 88.9)
- moved U1 52.7 mm to (56.9, 92.5), turned to 270 degrees
- moved R1 45.8 mm to (71.0, 96.0)
- moved D1 23.0 mm to (62.7, 116.1)
- moved D2 23.0 mm to (62.7, 113.5)
- moved D3 23.0 mm to (62.7, 111.0)
- moved R3 23.0 mm to (59.2, 116.3)
- moved R4 23.0 mm to (59.2, 113.8)
- moved R6 23.0 mm to (59.2, 111.3)
- moved U8 15.2 mm to (103.1, 72.6)
Connections:
- J8 pad 1: (no net) -> Net-(J8-Pad1)
- J8 pad 2: (no net) -> Net-(J8-Pad2)
- J8 pad 3: (no net) -> Net-(J8-Pad3)
- J8 pad 4: (no net) -> Net-(J8-Pad4)
- R3 pad 1: (no net) -> Net-(R3-Pad1)
- R4 pad 1: (no net) -> Net-(R4-Pad1)
- R6 pad 1: (no net) -> Net-(R6-Pad1)
- R7 pad 1: (no net) -> 3V3
- R8 pad 2: (no net) -> EN_ADDR8@FP2800A_5V
- U1 pad 1: (no net) -> SR2
- U1 pad 10: (no net) -> SRCLR_5V
- U1 pad 11: (no net) -> SRCLK_5V
- U1 pad 12: (no net) -> RCLK_5V
- U1 pad 14: (no net) -> SER_5V
- U1 pad 15: (no net) -> SR1
- U1 pad 2: (no net) -> SR3
- U1 pad 3: (no net) -> SR4
- U1 pad 4: (no net) -> SR5
- U1 pad 5: (no net) -> SR6
- U1 pad 6: (no net) -> SR7
- U1 pad 7: (no net) -> SR8
- U1 pad 9: (no net) -> Net-(U1-Pad9)

Commit message: update
Parts:
- removed J9: Conn_02x30_Odd_Even, Connector_PinHeader_2.54mm:PinHeader_2x30_P2.54mm_Vertical
- moved U2 154.0 mm to (-60.5, 44.7), turned to 90 degrees
- moved U1 142.2 mm to (-77.2, 45.2), turned to 90 degrees
- moved U8 127.1 mm to (19.8, -23.4)
- moved U5 125.5 mm to (-66.5, 61.5), turned to 90 degrees
- moved D1 116.8 mm to (8.86, 12.4)
- moved D3 116.8 mm to (8.86, 7.37)
- moved J1 116.8 mm to (16.3, 8.64)
- moved J2 116.8 mm to (20.3, 8.64)
- moved J3 116.8 mm to (24.4, 8.64)
- moved J4 116.8 mm to (28.4, 8.64)
- moved J5 116.8 mm to (53.3, -14.7)
- moved J6 116.8 mm to (53.3, -6.10)
- moved R1 116.8 mm to (17.2, -7.62)
- moved R4 116.8 mm to (5.36, 10.2)
- moved R5 116.8 mm to (42.7, -22.4)
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
Commit message: update
Parts:
- added U19: 5V_buck_converter, flipdot:5v_buck_converter, F.Cu at (81.3, 33.5)

Commit message: update
Parts:
- added J9: Barrel_Jack, Connector_BarrelJack:BarrelJack_Wuerth_6941xx301002, F.Cu at (193.0, 139.7)
- J7: moved to B.Cu
- moved U5 229.9 mm to (159.0, 106.0)
- moved U6 221.5 mm to (162.0, 120.0)
- moved U7 218.3 mm to (175.0, 118.0)
- moved U1 198.9 mm to (107.7, 118.6)
- moved U4 198.1 mm to (161.0, 95.0)
- moved U2 194.5 mm to (127.5, 94.7)
- moved U3 194.5 mm to (142.8, 94.2)
- moved U18 150.9 mm to (139.7, 74.9), turned to 0 degrees
- moved J8 150.8 mm to (109.0, 54.0)
- moved U16 150.6 mm to (177.0, 132.0), turned to 270 degrees
- moved C2 142.5 mm to (161.2, 59.7)
- moved C3 142.5 mm to (152.5, 59.7)
- moved C1 138.7 mm to (173.6, 35.5)
- moved D1 138.7 mm to (144.4, 41.9)
- moved D2 138.7 mm to (144.4, 39.4)
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Connections:
- U19 pad 1: (no net) -> 24V
- U19 pad 2: (no net) -> GND
- U19 pad 3: (no net) -> GND
- U19 pad 4: (no net) -> VCC
Routing:
- net 24V: track 0.00 -> 46.1 mm

Commit message: update
Parts:
- removed J2: 5V, Connector_PinHeader_2.54mm:PinHeader_1x02_P2.54mm_Vertical
- removed J3: 24V, Connector_PinHeader_2.54mm:PinHeader_1x02_P2.54mm_Vertical
- removed J4: EN_PWR, Connector_PinHeader_2.54mm:PinHeader_1x02_P2.54mm_Vertical
- removed J5, J6: Conn_01x02_Male, Connector_PinHeader_2.54mm:PinHeader_1x02_P2.54mm_Vertical
- added D4: D, Diode_THT:D_A-405_P7.62mm_Horizontal, F.Cu at (58.9, 118.1)
- added JP1: enable power rails, Connector_PinHeader_2.54mm:PinHeader_1x02_P2.54mm_Vertical, F.Cu at (68.8, 135.4)
- added JP2: current limited VS, Connector_PinHeader_2.54mm:PinHeader_1x02_P2.54mm_Vertical, F.Cu at (76.5, 135.4)
- added JP3: jumper 24v to display, Connector_PinHeader_2.54mm:PinHeader_1x02_P2.54mm_Vertical, F.Cu at (72.6, 135.4)
- added JP4: enable 5V VCC, Connector_PinHeader_2.54mm:PinHeader_1x02_P2.54mm_Vertical, F.Cu at (65.0, 135.4)
- J1: value 3V3 -> 3V3_from_wemos; footprint Connector_PinHeader_2.54mm:PinHeader_1x02_P2.54mm_Vertical -> Connector_PinHeader_2.54mm:PinHeader_1x01_P2.54mm_Vertical
- J8: value Conn_01x04 -> A0, D4, Rx, Tx
- R1, R5, U10, U11, U3, U4: moved to B.Cu
- U12, U13, U14: value A2982 -> TBD62783A
- U18: footprint Package_SO:SOP-20_7.5x12.8mm_P1.27mm -> Package_SO:SO-20_12.8x7.5mm_P1.27mm
- moved R7 167.1 mm to (41.5, 118.1)
- moved R1 166.4 mm to (39.4, 143.8), turned to 0 degrees
- moved R5 155.0 mm to (127.3, 153.4), turned to 270 degrees
- moved R8 153.9 mm to (40.4, 127.6), turned to 90 degrees
- moved U8 149.9 mm to (126.2, 153.2)
- moved R2 149.2 mm to (120.9, 153.2)
- moved J1 137.8 mm to (57.9, 138.9)
- moved R6 133.4 mm to (65.5, 147.1), turned to 90 degrees
- moved D3 132.4 mm to (65.5, 143.2), turned to 90 degrees
- moved R4 129.4 mm to (68.8, 147.1), turned to 90 degrees
- moved D2 128.4 mm to (68.8, 143.2), turned to 90 degrees
- moved R3 125.5 mm to (72.1, 147.1), turned to 90 degrees
- moved D1 124.4 mm to (72.1, 143.2), turned to 90 degrees
- moved C1 119.4 mm to (126.5, 145.3), turned to 0 degrees
- moved U3 118.4 mm to (41.9, 156.2), turned to 180 degrees
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Connections:
- net OE renamed ~OE
- net OE_5V renamed ~OE_5V
- net SRCLR renamed ~SRCLR
- net SRCLR_5V renamed ~SRCLR_5V
- C1 pad 1: Net-(C1-Pad1) -> 24V
- C2 pad 1: Net-(C1-Pad1) -> 24V
- J1 pad 1: 3V3 -> Net-(J1-Pad1)
- J7 pad 42: 24V -> 24V_to_display
- J7 pad 43: 24V -> 24V_to_display
- J7 pad 60: EN_ADDR8@FP2800A_24V -> (no net)
- R5 pad 2: Net-(C1-Pad1) -> 24V
- R7 pad 1: 3V3 -> ~EN_POWER_RAILS
- R7 pad 2: EN_POWER_RAILS -> Net-(D4-Pad1)
- R8 pad 1: VCC -> ~EN_ADDR8@FP2800A_5V
- R8 pad 2: EN_ADDR8@FP2800A_5V -> VCC
- U11 pad 5: (no net) -> GND
- U11 pad 6: (no net) -> GND
- U11 pad 7: (no net) -> GND
- U11 pad 8: (no net) -> GND
- U12 pad 1: (no net) -> GND
- U12 pad 10: (no net) -> GND
- U12 pad 11: (no net) -> SR17_ROW17_SET
- U12 pad 12: GND -> SR18_ROW18_SET
- U12 pad 13: SR17_ROW17_SET -> SR19_ROW19_SET
- U12 pad 14: SR18_ROW18_SET -> SR20_ROW20_SET
- U12 pad 15: SR19_ROW19_SET -> (no net)
- U12 pad 16: SR20_ROW20_SET -> (no net)
- U12 pad 3: (no net) -> Net-(U12-Pad3)
- U12 pad 4: (no net) -> Net-(U12-Pad3)
- U13 pad 10: (no net) -> GND
- U13 pad 11: (no net) -> SR9_ROW9_SET
- U13 pad 12: GND -> SR10_ROW10_SET
- U13 pad 13: SR9_ROW9_SET -> SR11_ROW11_SET
- U13 pad 14: SR10_ROW10_SET -> SR12_ROW12_SET
- U13 pad 15: SR11_ROW11_SET -> SR13_ROW13_SET
- U13 pad 16: SR12_ROW12_SET -> SR14_ROW14_SET
- U13 pad 17: SR13_ROW13_SET -> SR15_ROW15_SET
- U13 pad 18: SR14_ROW14_SET -> SR16_ROW16_SET
- U13 pad 19: SR15_ROW15_SET -> (no net)
- U13 pad 20: SR16_ROW16_SET -> (no net)
- U14 pad 10: (no net) -> GND
- U14 pad 11: (no net) -> SR1_ROW1_SET
- U14 pad 12: GND -> SR2_ROW2_SET
- U14 pad 13: SR1_ROW1_SET -> SR3_ROW3_SET
- U14 pad 14: SR2_ROW2_SET -> SR4_ROW4_SET
- U14 pad 15: SR3_ROW3_SET -> SR5_ROW5_SET
- U14 pad 16: SR4_ROW4_SET -> SR6_ROW6_SET
- U14 pad 17: SR5_ROW5_SET -> SR7_ROW7_SET
- U14 pad 18: SR6_ROW6_SET -> SR8_ROW8_SET
- U14 pad 19: SR7_ROW7_SET -> (no net)
- U14 pad 20: SR8_ROW8_SET -> (no net)
- U15 pad 12: EN_ADDR8@FP2800A -> ~EN_ADDR8@FP2800A
- U15 pad 14: EN_POWER_RAILS -> ~EN_POWER_RAILS
- U15 pad 8: 3V3 -> Net-(J1-Pad1)
- U15 pad 9: VCC -> Net-(D4-Pad1)
- U16 pad 1: EN_ADDR8@FP2800A_5V -> ~EN_ADDR8@FP2800A_5V
- U16 pad 18: EN_ADDR8@FP2800A_24V -> (no net)
- U16 pad 7: (no net) -> GND
- U16 pad 8: (no net) -> GND
- U18 pad 1: EN_POWER_RAILS -> ~EN_POWER_RAILS
- U18 pad 16: EN_ADDR8@FP2800A -> GND
- U18 pad 17: EN_ADDR8@FP2800A -> GND
- U18 pad 18: EN_ADDR8@FP2800A -> ~EN_ADDR8@FP2800A
- U18 pad 19: EN_POWER_RAILS -> ~EN_POWER_RAILS
- U18 pad 2: EN_ADDR8@FP2800A_5V -> ~EN_ADDR8@FP2800A_5V
- U18 pad 3: EN_ADDR8@FP2800A_5V -> (no net)
- U18 pad 4: EN_ADDR8@FP2800A_5V -> (no net)
- U19 pad 4: VCC -> Net-(JP4-Pad1)
- U8 pad 1: Net-(C1-Pad1) -> 24V
- U8 pad 4: EN_POWER_RAILS -> ~EN_POWER_RAILS
Routing:
- net VCC: track 0.00 -> 143.4 mm, vias 0 -> 5
- net ~EN_POWER_RAILS: track 0.00 -> 114.9 mm, vias 0 -> 6
- net VS: track 0.00 -> 99.8 mm, vias 0 -> 5
- net ~EN_ADDR8@FP2800A_5V: track 0.00 -> 94.5 mm, vias 0 -> 2
- net ~SRCLR_5V: track 0.00 -> 92.3 mm, vias 0 -> 5
- net 24V: track 46.1 -> 131.4 mm, vias 0 -> 1
- net Net-(C3-Pad1): track 0.00 -> 68.7 mm, vias 0 -> 1
- net SRCLK_5V: track 0.00 -> 59.6 mm, vias 0 -> 4
- net ~OE_5V: track 0.00 -> 58.9 mm, vias 0 -> 4
- net RCLK_5V: track 0.00 -> 56.7 mm, vias 0 -> 4
- net Net-(R6-Pad1): track 0.00 -> 50.7 mm, vias 0 -> 2
- net Net-(R4-Pad1): track 0.00 -> 48.7 mm, vias 0 -> 2
- net Net-(R3-Pad1): track 0.00 -> 47.4 mm, vias 0 -> 2
- net 24V_to_display: track 0.00 -> 43.1 mm
- net SR17: track 0.00 -> 33.3 mm, vias 0 -> 1
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- added copper zone on B.Cu, net GND
- added copper zone on F.Cu, net GND
Other:
- board size 100 x 100 mm -> 98 x 58.9 mm
