File: flipdot.sch (KiCad schematic (older format))
At the start: 41 parts, among them J1 3V3, J2 5V, J3 24V, J4 EN_PWR, J5 Conn_01x04_Female, J6 Conn_01x02_Male, J7 Conn_01x02_Male, J8 Conn_02x30_Odd_Even, U1 WeMos_D1_mini, U10 ULN2803A, U11 ULN2803A, U12 74HC595, U13 74HC595, U14 74HC595, U15 74HC595, U16 74HC595, U17 74HC595, U18 74HC595, U2 74HC245, U3 FPF2700, U4 ULN2803A, U5 ULN2803A, U6 TBD62783A, U7 TBD62783A, U8 TBD62783A, U9 ULN2803A

Commit message: update footprints
Parts:
- removed J5: Conn_01x04_Female, Connector_PinHeader_2.54mm:PinHeader_1x04_P2.54mm_Vertical, symbol Connector:Conn_01x04_Female
- added J8: Conn_01x04, Connector_PinHeader_2.54mm:PinHeader_1x04_P2.54mm_Vertical, symbol Connector_Generic:Conn_01x04
- J1, J2, J3, J4: footprint (none) -> Connector_PinHeader_2.54mm:PinHeader_1x02_P2.54mm_Vertical
- U1: renamed from U12; footprint (none) -> Package_SO:SOIC-16_3.9x9.9mm_P1.27mm
- U10, U11, U9: footprint (none) -> Package_SO:SOIC-18W_7.5x11.6mm_P1.27mm
- U15: renamed from U1; symbol wemos:WeMos_D1_mini -> flipdot-rescue:WeMos_D1_mini-wemos
- U16: renamed from U4; footprint (none) -> Package_SO:SOIC-18W_7.5x11.6mm_P1.27mm
- U17: renamed from U5; footprint (none) -> Package_SO:SOIC-18W_7.5x11.6mm_P1.27mm
- U18: renamed from U2; footprint (none) -> Package_SO:SOP-20_7.5x12.8mm_P1.27mm
- U2: renamed from U13; footprint (none) -> Package_SO:SOIC-16_3.9x9.9mm_P1.27mm
- U3: renamed from U14; footprint (none) -> Package_SO:SOIC-16_3.9x9.9mm_P1.27mm
- U4: renamed from U15; footprint (none) -> Package_SO:SOIC-16_3.9x9.9mm_P1.27mm
- U5: renamed from U16; footprint (none) -> Package_SO:SOIC-16_3.9x9.9mm_P1.27mm
- U6: renamed from U17; footprint (none) -> Package_SO:SOIC-16_3.9x9.9mm_P1.27mm
- U7: renamed from U18; footprint (none) -> Package_SO:SOIC-16_3.9x9.9mm_P1.27mm
- U8: renamed from U3; value FPF2700 -> FPF2702MX; symbol javl:FPF2700 -> flipdot:FPF2702MX
- gave numbers to parts that had none: 1
- renumbered J6 to J5, J7 to J6, J8 to J7, R5 to R1, R6 to R3, R7 to R4, R4 to R5, R8 to R6, R1 to R7, R3 to R8, U6 to U12, U7 to U13, U8 to U14
Connections:
- net labels added: SR21_ROW1_RST, SR22_ROW2_RST, SR23_ROW3_RST, SR24_ROW4_RST, SR25_ROW5_RST, SR26_ROW6_RST, SR27_ROW7_RST, SR28_ROW8_RST, SR29_ROW9_RST, SR30_ROW10_RST, SR31_ROW11_RST, SR32_ROW12_RST, SR33_ROW13_RST, SR34_ROW14_RST, SR35_ROW15_RST, SR36_ROW16_RST, SR37_ROW17_RST, SR38_ROW18_RST, SR39_ROW19_RST, SR40_ROW20_RST
- net labels removed: EN_ADD8@FP2800A_5V, OE_V5, SR21_ROW1_SET, SR21_ROW_1_RST, SR22_ROW2_SET, SR22_ROW_2_RST, SR23_ROW3_SET, SR23_ROW_3_RST, SR24_ROW4_SET, SR24_ROW_4_RST, SR25_ROW5_SET, SR25_ROW_5_RST, SR26_ROW6_SET, SR26_ROW_6_RST, SR27_ROW7_SET, SR27_ROW_7_RST, SR28_ROW8_SET, SR28_ROW_8_RST, SR29_ROW9_SET, SR29_ROW_9_RST, SR30_ROW10_SET, SR30_ROW_10_RST, SR31_ROW11_SET, SR31_ROW_11_RST, SR32_ROW12_SET, SR32_ROW_12_RST, SR33_ROW13_SET, SR33_ROW_13_RST, SR34_ROW14_SET, SR34_ROW_14_RST, SR35_ROW15_SET, SR35_ROW_15_RST, SR36_ROW16_SET, SR36_ROW_16_RST, SR37_ROW17_SET, SR37_ROW_17_RST, SR38_ROW18_SET, SR38_ROW_18_RST, SR39_ROW19_SET, SR39_ROW_19_RST, SR40_ROW20_SET, SR40_ROW_20_RST, SR48_ADDR1@FP2800A, SR54_LED_A, SR55_LED_B, SR56_LED_C, SR7_ROW_7_SET
- wire segments 531 -> 532
- no-connect marks 22 -> 23
Other:
- note added: "SR54_LED_A"
- note added: "SR55_LED_B"
- note added: "SR56_LED_C"
- moved on the sheet: R8

Commit message: update
Parts:
- removed U12, U13, U14: TBD62783A, symbol Transistor_Array:TBD62783A
- removed U15: WeMos_D1_mini, wemos:wemos-d1-mini-with-pin-header-and-connector, symbol flipdot-rescue:WeMos_D1_mini-wemos
- added U12, U13, U14: A2982, Package_SO:SOIC-20W_7.5x12.8mm_P1.27mm, symbol Transistor_Array:A2982
- added U15: WeMos_D1_mini, wemos:wemos-d1-mini-with-pin-header-and-connector, symbol Wemos_D1_Mini:WeMos_D1_mini
- C1: value 100u/35v -> 100uF/35v; footprint (none) -> Capacitor_SMD:CP_Elec_6.3x7.7
- C2: footprint (none) -> Capacitor_THT:CP_Radial_D6.3mm_P2.50mm
- C3: footprint (none) -> Capacitor_THT:CP_Radial_D5.0mm_P2.00mm
- D1: value LED C RED -> LED C; footprint LED_SMD:LED_0603_1608Metric -> LED_SMD:LED_0805_2012Metric
- D2: value LED B YELLOW -> LED B; footprint LED_SMD:LED_0603_1608Metric -> LED_SMD:LED_0805_2012Metric
- D3: value LED A GREEN -> LED A; footprint LED_SMD:LED_0603_1608Metric -> LED_SMD:LED_0805_2012Metric
- R1, R7, R8: footprint Resistor_SMD:R_0603_1608Metric -> Resistor_SMD:R_0805_2012Metric
- R4: value 150 -> 180
- R6: value 120 -> 180
Connections:
- net 3V3: now also U15.8 (3.3V)
- net EN_ADDR8@FP2800A: now also U15.12 (D3)
- net EN_POWER_RAILS: now also U15.14 (D1)
- net GND: now also U12.12 (GND), U13.12 (GND), U14.12 (GND), U15.10 (GND)
- net OE: now also U15.6 (D7)
- net RCLK: now also U15.5 (D6)
- net SER: now also U15.13 (D2)
- net SR1: now also U14.8 (IN8)
- net SR10: now also U13.7 (IN7)
- net SR10_ROW10_SET: now also U13.14 (OUT7)
- net SR11: now also U13.6 (IN6)
- net SR11_ROW11_SET: now also U13.15 (OUT6)
- net SR12: now also U13.5 (IN5)
- net SR12_ROW12_SET: now also U13.16 (OUT5)
- net SR13: now also U13.4 (IN4)
- net SR13_ROW13_SET: now also U13.17 (OUT4)
- net SR14: now also U13.3 (IN3)
- net SR14_ROW14_SET: now also U13.18 (OUT3)
- net SR15: now also U13.2 (IN2)
- net SR15_ROW15_SET: now also U13.19 (OUT2)
- net SR16: now also U13.1 (IN1)
- net SR16_ROW16_SET: now also U13.20 (OUT1)
- net SR17: now also U12.8 (IN8)
- net SR17_ROW17_SET: now also U12.13 (OUT8)
- net SR18: now also U12.7 (IN7)
- net SR18_ROW18_SET: now also U12.14 (OUT7)
- net SR19: now also U12.6 (IN6)
- net SR19_ROW19_SET: now also U12.15 (OUT6)
- net SR1_ROW1_SET: now also U14.13 (OUT8)
- net SR2: now also U14.7 (IN7)
- net SR20: now also U12.5 (IN5)
- net SR20_ROW20_SET: now also U12.16 (OUT5)
- net SR2_ROW2_SET: now also U14.14 (OUT7)
- net SR3: now also U14.6 (IN6)
- net SR3_ROW3_SET: now also U14.15 (OUT6)
- net SR4: now also U14.5 (IN5)
- net SR4_ROW4_SET: now also U14.16 (OUT5)
- net SR5: now also U14.4 (IN4)
- net SR5_ROW5_SET: now also U14.17 (OUT4)
- net SR6: now also U14.3 (IN3)
- net SR6_ROW6_SET: now also U14.18 (OUT3)
- net SR7: now also U14.2 (IN2)
- net SR7_ROW7_SET: now also U14.19 (OUT2)
- net SR8: now also U14.1 (IN1)
- net SR8_ROW8_SET: now also U14.20 (OUT1)
- net SR9: now also U13.8 (IN8)
- net SR9_ROW9_SET: now also U13.13 (OUT8)
- net SRCLK: now also U15.4 (D5)
- net SRCLR: now also U15.7 (D8)
- net VCC: now also U15.9 (5V)
- net VS: now also U12.9 (+VS), U13.9 (+VS), U14.9 (+VS)
- net at J8.1 (Pin_1): now also U15.2 (A0)
- net at J8.2 (Pin_2): now also U15.11 (D4)
- net at J8.3 (Pin_3): now also U15.15 (Rx)
- net at J8.4 (Pin_4): now also U15.16 (Tx)
- new net: U15.1 (Rst), U15.3 (D0)
Changed lines of the file:
@@
 P 2350 12050
 F 0 "D1" V 2297 12128 50  0000 L CNN
-F 1 "LED C RED" V 2388 12128 50  0000 L CNN
-F 2 "LED_SMD:LED_0603_1608Metric" H 2350 12050 50  0001 C CNN
+F 1 "LED C" V 2388 12128 50  0000 L CNN
+F 2 "LED_SMD:LED_0805_2012Metric" H 2350 12050 50  0001 C CNN
 F 3 "~" H 2350 12050 50  0001 C CNN
 	1    2350 12050
@@
 P 2900 11950
 F 0 "D2" V 2847 12028 50  0000 L CNN
-F 1 "LED B YELLOW" V 2938 12028 50  0000 L CNN
-F 2 "LED_SMD:LED_0603_1608Metric" H 2900 11950 50  0001 C CNN
+F 1 "LED B" V 2938 12028 50  0000 L CNN
+F 2 "LED_SMD:LED_0805_2012Metric" H 2900 11950 50  0001 C CNN
 F 3 "~" H 2900 11950 50  0001 C CNN
 	1    2900 11950
@@
 P 3450 11850
 F 0 "D3" V 3397 11929 50  0000 L CNN
-F 1 "LED A GREEN" V 3488 11929 50  0000 L CNN
-F 2 "LED_SMD:LED_0603_1608Metric" H 3450 11850 50  0001 C CNN
+F 1 "LED A" V 3488 11929 50  0000 L CNN
+F 2 "LED_SMD:LED_0805_2012Metric" H 3450 11850 50  0001 C CNN
 F 3 "~" H 3450 11850 50  0001 C CNN
 	1    3450 11850
@@
 P 2900 11650
 F 0 "R4" H 2970 11696 50  0000 L CNN
-F 1 "150" H 2970 11605 50  0000 L CNN
+F 1 "180" H 2970 11605 50  0000 L CNN
 F 2 "Resistor_SMD:R_0603_1608Metric" V 2830 11650 50  0001 C CNN
 F 3 "~" H 2900 11650 50  0001 C CNN
@@
 P 3450 11550
 F 0 "R6" H 3520 11596 50  0000 L CNN
-F 1 "120" H 3520 11505 50  0000 L CNN
+F 1 "180" H 3520 11505 50  0000 L CNN
 F 2 "Resistor_SMD:R_0603_1608Metric" V 3380 11550 50  0001 C CNN
 F 3 "~" H 3450 11550 50  0001 C CNN
@@
 F 0 "R1" V 1193 850 50  0000 C CNN
 F 1 "10K" V 1284 850 50  0000 C CNN
-F 2 "Resistor_SMD:R_0603_1608Metric" V 1330 850 50  0001 C CNN
+F 2 "Resistor_SMD:R_0805_2012Metric" V 1330 850 50  0001 C CNN
 F 3 "~" H 1400 850 50  0001 C CNN
 	1    1400 850
@@
 F 0 "R7" V 7657 5450 50  0000 C CNN
 F 1 "10K" V 7566 5450 50  0000 C CNN
-F 2 "Resistor_SMD:R_0603_1608Metric" V 7380 5450 50  0001 C CNN
+F 2 "Resistor_SMD:R_0805_2012Metric" V 7380 5450 50  0001 C CNN
 F 3 "~" H 7450 5450 50  0001 C CNN
 	1    7450 5450
@@
 Wire Wire Line
 	6950 5450 7300 5450
-Connection ~ 6950 5000
 Wire Wire Line
 	8000 4500 8000 5450
@@
 Wire Wire Line
 	8100 4300 7950 4300
-$Comp
-L flipdot-rescue:WeMos_D1_mini-wemos U15
-U 1 1 63B544EE
-P 7450 4650
-F 0 "U15" H 7450 5287 60  0000 C CNN
-F 1 "WeMos_D1_mini" H 7450 5181 60  0000 C CNN
-F 2 "wemos:wemos-d1-mini-with-pin-header-and-connector" H 7450 5181 60  0001 C CNN
-F 3 "http://www.wemos.cc/Products/d1_mini.html" H 7450 5181 60  0001 C CNN
-	1    7450 4650
-	1    0    0    -1
-$EndComp
 Wire Notes Line
 	600  500  600  12300
@@
 F 0 "C3" H 3665 14246 50  0000 L CNN
 F 1 "22u" H 3665 14155 50  0000 L CNN
-F 2 "" H 3588 14050 50  0001 C CNN
+F 2 "Capacitor_THT:CP_Radial_D5.0mm_P2.00mm" H 3588 14050 50  0001 C CNN
 F 3 "~" H 3550 14200 50  0001 C CNN
 	1    3550 14200
@@
 P 1550 14150
 F 0 "C1" H 1432 14104 50  0000 R CNN
-F 1 "100u/35v" H 1432 14195 50  0000 R CNN
-F 2 "" H 1588 14000 50  0001 C CNN
+F 1 "100uF/35v" H 1432 14195 50  0000 R CNN
+F 2 "Capacitor_SMD:CP_Elec_6.3x7.7" H 1588 14000 50  0001 C CNN
 F 3 "~" H 1550 14150 50  0001 C CNN
 	1    1550 14150
@@
 F 0 "C2" H 1915 14196 50  0000 L CNN
 F 1 "100u" H 1915 14105 50  0000 L CNN
-F 2 "" H 1838 14000 50  0001 C CNN
+F 2 "Capacitor_THT:CP_Radial_D6.3mm_P2.50mm" H 1838 14000 50  0001 C CNN
 F 3 "~" H 1800 14150 50  0001 C CNN
 	1    1800 14150
@@
 	1    0    0    -1
 $EndComp
-$Comp
-L Transistor_Array:TBD62783A U12
-U 1 1 610D9792
-P 5050 6250
-F 0 "U12" H 5050 6931 50  0000 C CNN
-F 1 "TBD62783A" H 5050 6840 50  0000 C CNN
-F 2 "" H 5050 5700 50  0001 C CNN
-F 3 "http://toshiba.semicon-storage.com/info/docget.jsp?did=30523&prodName=TBD62783APG" H 4750 6650 50  0001 C CNN
-	1    5050 6250
-	1    0    0    -1
-$EndComp
 Wire Wire Line
 	4900 7400 5050 7400
@@
 	1    0    0    -1
 $EndComp
-$Comp
-L Transistor_Array:TBD62783A U13
-U 1 1 6109BC93
-P 5050 7900
-F 0 "U13" H 5050 8581 50  0000 C CNN
-F 1 "TBD62783A" H 5050 8490 50  0000 C CNN
-F 2 "" H 5050 7350 50  0001 C CNN
-F 3 "http://toshiba.semicon-storage.com/info/docget.jsp?did=30523&prodName=TBD62783APG" H 4750 8300 50  0001 C CNN
-	1    5050 7900
-	1    0    0    -1
-$EndComp
 Text GLabel 4900 9050 0    50   Input ~ 0
 VS
@@
 	1    0    0    -1
 $EndComp
-$Comp
-L Transistor_Array:TBD62783A U14
-U 1 1 60CEAA19
-P 5050 9550
-F 0 "U14" H 5050 10231 50  0000 C CNN
-F 1 "TBD62783A" H 5050 10140 50  0000 C CNN
-F 2 "" H 5050 9000 50  0001 C CNN
-F 3 "http://toshiba.semicon-storage.com/info/docget.jsp?did=30523&prodName=TBD62783APG" H 4750 9950 50  0001 C CNN
-	1    5050 9550
-	1    0    0    -1
-$EndComp
 Wire Notes Line
 	4250 5400 4250 10400
@@
 F 0 "R8" V 8293 7700 50  0000 C CNN
 F 1 "10K" V 8384 7700 50  0000 C CNN
-F 2 "Resistor_SMD:R_0603_1608Metric" V 8430 7700 50  0001 C CNN
+F 2 "Resistor_SMD:R_0805_2012Metric" V 8430 7700 50  0001 C CNN
 F 3 "~" H 8500 7700 50  0001 C CNN
 	1    8500 7700
@@
 	1    0    0    -1
 $EndComp
+$Comp
+L Transistor_Array:A2982 U14
+U 1 1 5F9072C4
+P 5050 9550
+F 0 "U14" H 5050 10231 50  0000 C CNN
+F 1 "A2982" H 5050 10140 50  0000 C CNN
+F 2 "Package_SO:SOIC-20W_7.5x12.8mm_P1.27mm" H 5050 9000 50  0001 C CNN
+F 3 "https://www.allegromicro.com/~/media/Files/Datasheets/A2981-2-Datasheet.ashx" H 4750 9950 50  0001 C CNN
+	1    5050 9550
+	1    0    0    -1
+$EndComp
+$Comp
+L Transistor_Array:A2982 U13
+U 1 1 5F908136
+P 5050 7900
+F 0 "U13" H 5050 8581 50  0000 C CNN
+F 1 "A2982" H 5050 8490 50  0000 C CNN
+F 2 "Package_SO:SOIC-20W_7.5x12.8mm_P1.27mm" H 5050 7350 50  0001 C CNN
+F 3 "https://www.allegromicro.com/~/media/Files/Datasheets/A2981-2-Datasheet.ashx" H 4750 8300 50  0001 C CNN
+	1    5050 7900
+	1    0    0    -1
+$EndComp
+$Comp
+L Transistor_Array:A2982 U12
+U 1 1 5F908AE5
+P 5050 6250
+F 0 "U12" H 5050 6931 50  0000 C CNN
+F 1 "A2982" H 5050 6840 50  0000 C CNN
+F 2 "Package_SO:SOIC-20W_7.5x12.8mm_P1.27mm" H 5050 5700 50  0001 C CNN
+F 3 "https://www.allegromicro.com/~/media/Files/Datasheets/A2981-2-Datasheet.ashx" H 4750 6650 50  0001 C CNN
+	1    5050 6250
+	1    0    0    -1
+$EndComp
+$Comp
+L Wemos_D1_Mini:WeMos_D1_mini U15
+U 1 1 5F8C5DFE
+P 7450 4650
+F 0 "U15" H 7450 5287 60  0000 C CNN
+F 1 "WeMos_D1_mini" H 7450 5181 60  0000 C CNN
+F 2 "wemos:wemos-d1-mini-with-pin-header-and-connector" H 8000 3950 60  0000 C CNN
+F 3 "http://www.wemos.cc/Products/d1_mini.html" H 7450 5181 60  0001 C CNN
+	1    7450 4650
+	1    0    0    -1
+$EndComp
+Connection ~ 6950 5000
 $EndSCHEMATC

Commit message: update
Parts:
- removed J9: Conn_02x30_Odd_Even, Connector_PinHeader_2.54mm:PinHeader_2x30_P2.54mm_Vertical, symbol Connector_Generic:Conn_02x30_Odd_Even
Connections:
- no-connect marks 23 -> 22
Other:
- note removed: "60-pol BROSE connector (#2 for daisy chaining)"
- moved on the sheet: J7

Commit message: update
Parts:
- added U19: 5V_buck_converter, flipdot:5v_buck_converter, symbol flipdot:5V_buck_converter
Changed lines of the file:
@@
 $EndComp
 Connection ~ 6950 5000
+$Comp
+L flipdot:5V_buck_converter U19
+U 1 1 5F9259D9
+P 5450 11150
+F 0 "U19" H 5375 11175 50  0000 C CNN
+F 1 "5V_buck_converter" H 5375 11084 50  0000 C CNN
+F 2 "flipdot:5v_buck_converter" H 5450 11150 50  0001 C CNN
+F 3 "" H 5450 11150 50  0001 C CNN
+	1    5450 11150
+	1    0    0    -1
+$EndComp
 $EndSCHEMATC

Commit message: update
Parts:
- added J9: Barrel_Jack, Connector_BarrelJack:BarrelJack_Wuerth_6941xx301002, symbol Connector:Barrel_Jack
Connections:
- net 24V: now also U19.1 (in+), J9.1
- net GND: now also U19.2 (in-), U19.3 (out-), J9.2
- net VCC: now also U19.4 (out+)
Other:
- note added: "Power Supply In and to 5V (VCC)"
- moved on the sheet: U19
Changed lines of the file:
@@
 L flipdot:5V_buck_converter U19
 U 1 1 5F9259D9
-P 5450 11150
-F 0 "U19" H 5375 11175 50  0000 C CNN
-F 1 "5V_buck_converter" H 5375 11084 50  0000 C CNN
-F 2 "flipdot:5v_buck_converter" H 5450 11150 50  0001 C CNN
-F 3 "" H 5450 11150 50  0001 C CNN
-	1    5450 11150
+P 6250 13150
+F 0 "U19" H 6175 13175 50  0000 C CNN
+F 1 "5V_buck_converter" H 6175 13084 50  0000 C CNN
+F 2 "flipdot:5v_buck_converter" H 6250 13150 50  0001 C CNN
+F 3 "" H 6250 13150 50  0001 C CNN
+	1    6250 13150
 	1    0    0    -1
 $EndComp
+Text GLabel 5700 13250 1    50   Input ~ 0
+24V
+$Comp
+L power:GND #PWR0104
+U 1 1 5F93A3EF
+P 6200 13850
+F 0 "#PWR0104" H 6200 13600 50  0001 C CNN
+F 1 "GND" H 6205 13677 50  0000 C CNN
+F 2 "" H 6200 13850 50  0001 C CNN
+F 3 "" H 6200 13850 50  0001 C CNN
+	1    6200 13850
+	1    0    0    -1
+$EndComp
+Wire Wire Line
+	5800 13550 5700 13550
+Wire Wire Line
+	5700 13550 5700 13750
+Wire Wire Line
+	5700 13750 6200 13750
+Wire Wire Line
+	6700 13750 6700 13550
+Wire Wire Line
+	6700 13550 6600 13550
+Wire Wire Line
+	6200 13850 6200 13750
+Connection ~ 6200 13750
+Wire Wire Line
+	6200 13750 6700 13750
+Text GLabel 6700 13350 2    50   Output ~ 0
+VCC
+Wire Wire Line
+	6700 13350 6600 13350
+Wire Wire Line
+	5400 13350 5700 13350
+Wire Wire Line
+	5700 13250 5700 13350
+Connection ~ 5700 13350
+Wire Wire Line
+	5700 13350 5800 13350
+Wire Wire Line
+	5400 13550 5700 13550
+Connection ~ 5700 13550
+Wire Notes Line
+	3900 12800 6950 12800
+Wire Notes Line
+	6950 12800 6950 14150
+Wire Notes Line
+	6950 14150 3900 14150
+Wire Notes Line
+	3900 14150 3900 12800
+Text Notes 3950 12900 0    50   ~ 0
+Power Supply In and to 5V (VCC)
+$Comp
+L Connector:Barrel_Jack J9
+U 1 1 5FFB73BB
+P 5100 13450
+F 0 "J9" H 5157 13775 50  0000 C CNN
+F 1 "Barrel_Jack" H 5157 13684 50  0000 C CNN
+F 2 "Connector_BarrelJack:BarrelJack_Wuerth_6941xx301002" H 5150 13410 50  0001 C CNN
+F 3 "~" H 5150 13410 50  0001 C CNN
+	1    5100 13450
+	1    0    0    -1
+$EndComp

Commit message: update
Parts:
- removed J1: 3V3, Connector_PinHeader_2.54mm:PinHeader_1x02_P2.54mm_Vertical, symbol Connector:Conn_01x02_Male
- removed J2: 5V, Connector_PinHeader_2.54mm:PinHeader_1x02_P2.54mm_Vertical, symbol Connector:Conn_01x02_Male
- removed J3: 24V, Connector_PinHeader_2.54mm:PinHeader_1x02_P2.54mm_Vertical, symbol Connector:Conn_01x02_Male
- removed J4: EN_PWR, Connector_PinHeader_2.54mm:PinHeader_1x02_P2.54mm_Vertical, symbol Connector:Conn_01x02_Male
- removed J5, J6: Conn_01x02_Male, Connector_PinHeader_2.54mm:PinHeader_1x02_P2.54mm_Vertical, symbol Connector:Conn_01x02_Male
- removed U12, U13, U14: A2982, Package_SO:SOIC-20W_7.5x12.8mm_P1.27mm, symbol Transistor_Array:A2982
- added D4: D, Diode_THT:D_A-405_P7.62mm_Horizontal, symbol Device:D
- added J1: 3V3_from_wemos, Connector_PinHeader_2.54mm:PinHeader_1x01_P2.54mm_Vertical, symbol Connector:Conn_01x01_Female
- added JP1: enable power rails, Connector_PinHeader_2.54mm:PinHeader_1x02_P2.54mm_Vertical, symbol Device:Jumper_NC_Small
- added JP2: current limited VS, Connector_PinHeader_2.54mm:PinHeader_1x02_P2.54mm_Vertical, symbol Device:Jumper_NC_Small
- added JP3: jumper 24v to display, Connector_PinHeader_2.54mm:PinHeader_1x02_P2.54mm_Vertical, symbol Device:Jumper_NC_Small
- added JP4: enable 5V VCC, Connector_PinHeader_2.54mm:PinHeader_1x02_P2.54mm_Vertical, symbol Device:Jumper_NC_Small
- added U12, U13, U14: TBD62783A, Package_SO:SOIC-20W_7.5x12.8mm_P1.27mm, symbol Transistor_Array:TBD62783A
- J8: value Conn_01x04 -> A0, D4, Rx, Tx
- U15: symbol Wemos_D1_Mini:WeMos_D1_mini -> flipdot-rescue:WeMos_D1_mini-Wemos_D1_Mini
- U18: footprint Package_SO:SOP-20_7.5x12.8mm_P1.27mm -> Package_SO:SO-20_12.8x7.5mm_P1.27mm
Connections:
- net 24V: now also C1.1, C2.1, R5.2, U8.1 (VIN), JP3.1; no longer J7.42 (Pin_42), J7.43 (Pin_43)
- net EN_ADDR8@FP2800A_24V: no longer U16.18 (O1)
- net GND: now also U11.5 (I5), U11.6 (I6), U11.7 (I7), U11.8 (I8), U16.7 (I7), U16.8 (I8), U18.16 (B2), U18.17 (B1), JP1.2, U12.1 (I1), U12.10 (GND), U12.2 (I2), U12.3 (I3), U12.4 (I4), U13.10 (GND), U14.10 (GND)
- net SR1: now also U14.8 (I8)
- net SR10: now also U13.7 (I7)
- net SR10_ROW10_SET: now also U13.12 (O7)
- net SR11: now also U13.6 (I6)
- net SR11_ROW11_SET: now also U13.13 (O6)
- net SR12: now also U13.5 (I5)
- net SR12_ROW12_SET: now also U13.14 (O5)
- net SR13: now also U13.4 (I4)
- net SR13_ROW13_SET: now also U13.15 (O4)
- net SR14: now also U13.3 (I3)
- net SR14_ROW14_SET: now also U13.16 (O3)
- net SR15: now also U13.2 (I2)
- net SR15_ROW15_SET: now also U13.17 (O2)
- net SR16: now also U13.1 (I1)
- net SR16_ROW16_SET: now also U13.18 (O1)
- net SR17: now also U12.8 (I8)
- net SR17_ROW17_SET: now also U12.11 (O8)
- net SR18: now also U12.7 (I7)
- net SR18_ROW18_SET: now also U12.12 (O7)
- net SR19: now also U12.6 (I6)
- net SR19_ROW19_SET: now also U12.13 (O6)
- net SR1_ROW1_SET: now also U14.11 (O8)
- net SR2: now also U14.7 (I7)
- net SR20: now also U12.5 (I5)
- net SR20_ROW20_SET: now also U12.14 (O5)
- net SR2_ROW2_SET: now also U14.12 (O7)
- net SR3: now also U14.6 (I6)
- net SR3_ROW3_SET: now also U14.13 (O6)
- net SR4: now also U14.5 (I5)
- net SR4_ROW4_SET: now also U14.14 (O5)
- net SR5: now also U14.4 (I4)
- net SR5_ROW5_SET: now also U14.15 (O4)
- net SR6: now also U14.3 (I3)
- net SR6_ROW6_SET: now also U14.16 (O3)
- net SR7: now also U14.2 (I2)
- net SR7_ROW7_SET: now also U14.17 (O2)
- net SR8: now also U14.1 (I1)
- net SR8_ROW8_SET: now also U14.18 (O1)
- net SR9: now also U13.8 (I8)
- net SR9_ROW9_SET: now also U13.11 (O8)
- net VCC: now also R8.2, D4.2 (A), JP4.2; no longer R8.1, U15.9 (5V), U19.4 (out+)
- net VS: now also JP2.1, U12.9 (VCC), U13.9 (VCC), U14.9 (VCC)
- net at C3.1, U8.8 (VOUT): now also JP2.2
- net 3V3: no longer names the net of U15.8 (3.3V)
- net 3V3: now also J1.1 (Pin_1); no longer R7.1
- net EN_ADDR8@FP2800A renamed ~EN_ADDR8@FP2800A
- net ~EN_ADDR8@FP2800A: no longer U18.16 (B2), U18.17 (B1)
- removed net EN_ADDR8@FP2800A_5V: R8.2, U16.1 (I1), U18.2 (A0), U18.3 (A1), U18.4 (A2)
- net EN_POWER_RAILS renamed ~EN_POWER_RAILS
- net ~EN_POWER_RAILS: now also R7.1, JP1.1; no longer R7.2
- net OE renamed ~OE
- net OE_5V renamed ~OE_5V
- net SRCLR renamed ~SRCLR
- net SRCLR_5V renamed ~SRCLR_5V
- new net: D4.1 (K), R7.2, U15.9 (5V)
- new net: JP4.1, U19.4 (out+)
- new net 24V_to_display: J7.42 (Pin_42), J7.43 (Pin_43), JP3.2
- new net ~EN_ADDR8@FP2800A_24V: U16.18 (O1)
- new net ~EN_ADDR8@FP2800A_5V: R8.1, U16.1 (I1), U18.2 (A0)
- no-connect marks 22 -> 14
Other:
- moved on the sheet: C1, C2, C3, J8, J9, R2, R5, R7, R8, U15, U17, U18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
