File: flipdot.sch (KiCad schematic (older format))
At the start: 42 parts, among them J1 3V3_from_wemos, J7 Conn_02x30_Odd_Even, J8 A0, D4, Rx, Tx, J9 Barrel_Jack, U1 74HC595, U10 ULN2803A, U11 ULN2803A, U12 TBD62783A, U13 TBD62783A, U14 TBD62783A, U15 WeMos_D1_mini, U16 ULN2803A, U17 ULN2803A, U18 74HC245, U19 5V_buck_converter, U2 74HC595, U3 74HC595, U4 74HC595, U5 74HC595, U6 74HC595, U7 74HC595, U8 FPF2702MX, U9 ULN2803A

Commit message: update
Parts:
- D4: footprint Diode_THT:D_A-405_P7.62mm_Horizontal -> Diode_THT:D_DO-35_SOD27_P7.62mm_Horizontal
- J8: value A0, D4, Rx, Tx -> A0 D4 Rx Tx
- JP1, JP2, JP3, JP4: footprint Connector_PinHeader_2.54mm:PinHeader_1x02_P2.54mm_Vertical -> javl:PinHeader_1x02_P2.54mm_Vertical-No-Markings
- R1, R7, R8: footprint Resistor_SMD:R_0805_2012Metric -> Resistor_SMD:R_0805_2012Metric_Pad1.20x1.40mm_HandSolder
- R2, R3, R4, R5, R6: footprint Resistor_SMD:R_0603_1608Metric -> Resistor_SMD:R_0805_2012Metric_Pad1.20x1.40mm_HandSolder
- U18: footprint Package_SO:SO-20_12.8x7.5mm_P1.27mm -> Package_SO:SO-20_5.3x12.6mm_P1.27mm
Connections:
- net at J1.1 (Pin_1), U15.8 (3.3V): now also R7.2
- net at D4.1 (K), U15.9 (5V): no longer R7.2
Changed lines of the file:
@@
 F 0 "R3" H 2420 11796 50  0000 L CNN
 F 1 "180" H 2420 11705 50  0000 L CNN
-F 2 "Resistor_SMD:R_0603_1608Metric" V 2280 11750 50  0001 C CNN
+F 2 "Resistor_SMD:R_0805_2012Metric_Pad1.20x1.40mm_HandSolder" V 2280 11750 50  0001 C CNN
 F 3 "~" H 2350 11750 50  0001 C CNN
 	1    2350 11750
@@
 F 0 "R4" H 2970 11696 50  0000 L CNN
 F 1 "180" H 2970 11605 50  0000 L CNN
-F 2 "Resistor_SMD:R_0603_1608Metric" V 2830 11650 50  0001 C CNN
+F 2 "Resistor_SMD:R_0805_2012Metric_Pad1.20x1.40mm_HandSolder" V 2830 11650 50  0001 C CNN
 F 3 "~" H 2900 11650 50  0001 C CNN
 	1    2900 11650
@@
 F 0 "R6" H 3520 11596 50  0000 L CNN
 F 1 "180" H 3520 11505 50  0000 L CNN
-F 2 "Resistor_SMD:R_0603_1608Metric" V 3380 11550 50  0001 C CNN
+F 2 "Resistor_SMD:R_0805_2012Metric_Pad1.20x1.40mm_HandSolder" V 3380 11550 50  0001 C CNN
 F 3 "~" H 3450 11550 50  0001 C CNN
 	1    3450 11550
@@
 F 0 "R1" V 1193 850 50  0000 C CNN
 F 1 "10K" V 1284 850 50  0000 C CNN
-F 2 "Resistor_SMD:R_0805_2012Metric" V 1330 850 50  0001 C CNN
+F 2 "Resistor_SMD:R_0805_2012Metric_Pad1.20x1.40mm_HandSolder" V 1330 850 50  0001 C CNN
 F 3 "~" H 1400 850 50  0001 C CNN
 	1    1400 850
@@
 F 0 "R7" V 9207 4850 50  0000 C CNN
 F 1 "10K" V 9116 4850 50  0000 C CNN
-F 2 "Resistor_SMD:R_0805_2012Metric" V 8930 4850 50  0001 C CNN
+F 2 "Resistor_SMD:R_0805_2012Metric_Pad1.20x1.40mm_HandSolder" V 8930 4850 50  0001 C CNN
 F 3 "~" H 9000 4850 50  0001 C CNN
 	1    9000 4850
@@
 F 0 "R2" H 1920 13946 50  0000 L CNN
 F 1 "470K" H 1920 13855 50  0000 L CNN
-F 2 "Resistor_SMD:R_0603_1608Metric" V 1780 13900 50  0001 C CNN
+F 2 "Resistor_SMD:R_0805_2012Metric_Pad1.20x1.40mm_HandSolder" V 1780 13900 50  0001 C CNN
 F 3 "~" H 1850 13900 50  0001 C CNN
 	1    1850 13900
@@
 F 0 "R5" V 3207 13100 50  0000 C CNN
 F 1 "100K" V 3116 13100 50  0000 C CNN
-F 2 "Resistor_SMD:R_0603_1608Metric" V 2930 13100 50  0001 C CNN
+F 2 "Resistor_SMD:R_0805_2012Metric_Pad1.20x1.40mm_HandSolder" V 2930 13100 50  0001 C CNN
 F 3 "~" H 3000 13100 50  0001 C CNN
 	1    3000 13100
@@
 F 0 "R8" V 8143 7750 50  0000 C CNN
 F 1 "10K" V 8234 7750 50  0000 C CNN
-F 2 "Resistor_SMD:R_0805_2012Metric" V 8280 7750 50  0001 C CNN
+F 2 "Resistor_SMD:R_0805_2012Metric_Pad1.20x1.40mm_HandSolder" V 8280 7750 50  0001 C CNN
 F 3 "~" H 8350 7750 50  0001 C CNN
 	1    8350 7750
@@
 F 0 "U18" H 8000 5919 50  0000 C CNN
 F 1 "74HC245" H 8000 6010 50  0000 C CNN
-F 2 "Package_SO:SO-20_12.8x7.5mm_P1.27mm" H 8000 6900 50  0001 C CNN
+F 2 "Package_SO:SO-20_5.3x12.6mm_P1.27mm" H 8000 6900 50  0001 C CNN
 F 3 "http://www.ti.com/lit/gpn/sn74HC245" H 8000 6900 50  0001 C CNN
 	1    8000 6900
@@
 P 9000 4150
 F 0 "J8" H 9080 4142 50  0000 L CNN
-F 1 "A0, D4, Rx, Tx" H 9080 4051 50  0000 L CNN
+F 1 "A0 D4 Rx Tx" H 9080 4051 50  0000 L CNN
 F 2 "Connector_PinHeader_2.54mm:PinHeader_1x04_P2.54mm_Vertical" H 9000 4150 50  0001 C CNN
 F 3 "~" H 9000 4150 50  0001 C CNN
@@
 F 0 "D4" H 8300 5316 50  0000 C CNN
 F 1 "D" H 8300 5225 50  0000 C CNN
-F 2 "Diode_THT:D_A-405_P7.62mm_Horizontal" H 8300 5100 50  0001 C CNN
+F 2 "Diode_THT:D_DO-35_SOD27_P7.62mm_Horizontal" H 8300 5100 50  0001 C CNN
 F 3 "~" H 8300 5100 50  0001 C CNN
 	1    8300 5100
@@
 	6950 5200 7150 5200
 Wire Wire Line
-	9000 5000 8150 5000
-Connection ~ 8150 5000
-Wire Wire Line
 	8500 5100 8450 5100
 NoConn ~ 8500 7300
@@
 F 0 "JP2" H 2900 12962 50  0000 C CNN
 F 1 "current limited VS" H 2900 12850 50  0000 C CNN
-F 2 "Connector_PinHeader_2.54mm:PinHeader_1x02_P2.54mm_Vertical" H 2900 12750 50  0001 C CNN
+F 2 "javl:PinHeader_1x02_P2.54mm_Vertical-No-Markings" H 2900 12750 50  0001 C CNN
 F 3 "~" H 2900 12750 50  0001 C CNN
 	1    2900 12750
@@
 F 0 "JP1" H 2850 14812 50  0000 C CNN
 F 1 "enable power rails" H 2850 14700 50  0000 C CNN
-F 2 "Connector_PinHeader_2.54mm:PinHeader_1x02_P2.54mm_Vertical" H 2850 14600 50  0001 C CNN
+F 2 "javl:PinHeader_1x02_P2.54mm_Vertical-No-Markings" H 2850 14600 50  0001 C CNN
 F 3 "~" H 2850 14600 50  0001 C CNN
 	1    2850 14600
@@
 F 0 "JP3" H 5400 13112 50  0000 C CNN
 F 1 "jumper 24v to display" H 5400 13000 50  0000 C CNN
-F 2 "Connector_PinHeader_2.54mm:PinHeader_1x02_P2.54mm_Vertical" H 5400 12900 50  0001 C CNN
+F 2 "javl:PinHeader_1x02_P2.54mm_Vertical-No-Markings" H 5400 12900 50  0001 C CNN
 F 3 "~" H 5400 12900 50  0001 C CNN
 	1    5400 12900
@@
 F 0 "JP4" H 5800 13412 50  0000 C CNN
 F 1 "enable 5V VCC" H 5800 13300 50  0000 C CNN
-F 2 "Connector_PinHeader_2.54mm:PinHeader_1x02_P2.54mm_Vertical" H 5800 13200 50  0001 C CNN
+F 2 "javl:PinHeader_1x02_P2.54mm_Vertical-No-Markings" H 5800 13200 50  0001 C CNN
 F 3 "~" H 5800 13200 50  0001 C CNN
 	1    5800 13200
@@
 	5400 13200 5700 13200
 Wire Wire Line
-	9900 14650 10100 14650
+	9900 14650 10000 14650
 Wire Wire Line
 	4650 6050 4650 5950
@@
 	2150 13400 1400 13400
 Connection ~ 1400 13400
+Wire Wire Line
+	7150 5200 9000 5200
+Wire Wire Line
+	9000 5200 9000 5000
+Connection ~ 7150 5200
 $EndSCHEMATC

Commit message: update
Parts:
- U12, U13, U14: footprint Package_SO:SOIC-20W_7.5x12.8mm_P1.27mm -> Package_SO:SOIC-18W_7.5x11.6mm_P1.27mm
Changed lines of the file:
@@
 F 0 "U14" H 5050 10231 50  0000 C CNN
 F 1 "TBD62783A" H 5050 10140 50  0000 C CNN
-F 2 "Package_SO:SOIC-20W_7.5x12.8mm_P1.27mm" H 5050 9000 50  0001 C CNN
+F 2 "Package_SO:SOIC-18W_7.5x11.6mm_P1.27mm" H 5050 9000 50  0001 C CNN
 F 3 "http://toshiba.semicon-storage.com/info/docget.jsp?did=30523&prodName=TBD62783APG" H 4750 9950 50  0001 C CNN
 	1    5050 9550
@@
 F 0 "U13" H 5050 8581 50  0000 C CNN
 F 1 "TBD62783A" H 5050 8490 50  0000 C CNN
-F 2 "Package_SO:SOIC-20W_7.5x12.8mm_P1.27mm" H 5050 7350 50  0001 C CNN
+F 2 "Package_SO:SOIC-18W_7.5x11.6mm_P1.27mm" H 5050 7350 50  0001 C CNN
 F 3 "http://toshiba.semicon-storage.com/info/docget.jsp?did=30523&prodName=TBD62783APG" H 4750 8300 50  0001 C CNN
 	1    5050 7900
@@
 F 0 "U12" H 5050 6931 50  0000 C CNN
 F 1 "TBD62783A" H 5050 6840 50  0000 C CNN
-F 2 "Package_SO:SOIC-20W_7.5x12.8mm_P1.27mm" H 5050 5700 50  0001 C CNN
+F 2 "Package_SO:SOIC-18W_7.5x11.6mm_P1.27mm" H 5050 5700 50  0001 C CNN
 F 3 "http://toshiba.semicon-storage.com/info/docget.jsp?did=30523&prodName=TBD62783APG" H 4750 6650 50  0001 C CNN
 	1    5050 6250
