File: flipdot_compact.kicad_pcb (KiCad board)
At the start: 2 copper layers, 100 x 49.3 mm, 47 parts, among them J1 3V3_from_wemos, J7 Conn_02x30_Odd_Even, J8 A0 D4 Rx Tx, J9 Barrel_Jack, U1 74HC595, U10 ULN2803A, U11 ULN2803A, U12 TBD62783A, U13 TBD62783A, U14 TBD62783A, U15 WeMos_D1_mini, U16 ULN2803A, U17 ULN2803A, U18 74HC245, U19 5V_buck_converter, U2 74HC595, U3 74HC595, U4 74HC595, U5 74HC595, U6 74HC595, U7 74HC595, U8 FPF2702MX, U9 ULN2803A

Commit message: update
Other:
- board text added: "JLCJLCJLCJLC"

Commit message: update
Parts:
- U12, U13, U14: footprint Package_SO:SOIC-20W_7.5x12.8mm_P1.27mm -> Package_SO:SOIC-18W_7.5x11.6mm_P1.27mm
- moved U12 1.00 mm to (72.6, 158.5)
- moved U13 1.00 mm to (57.7, 158.5)
- moved U14 1.00 mm to (42.7, 158.5)
- moved U17 1.00 mm to (100.8, 158.5)
- moved U9 1.00 mm to (87.1, 158.5)
Routing:
- net GND: track 375.8 -> 0.00 mm, vias 4 -> 0
- net VCC: track 227.6 -> 0.00 mm, vias 3 -> 0
- net VS: track 165.0 -> 0.00 mm, vias 2 -> 0
- net ~OE_5V: track 153.0 -> 0.00 mm, vias 5 -> 0
- net RCLK_5V: track 151.0 -> 0.00 mm, vias 5 -> 0
- net ~SRCLR_5V: track 148.5 -> 0.00 mm, vias 4 -> 0
- net SRCLK_5V: track 146.0 -> 0.00 mm, vias 5 -> 0
- net ~EN_POWER_RAILS: track 119.9 -> 0.00 mm
- net 24V: track 118.0 -> 0.00 mm
- net 24V_to_display: track 107.4 -> 0.00 mm
- net ~EN_ADDR8@FP2800A_5V: track 80.0 -> 0.00 mm
- net Net-(C3-Pad1): track 66.1 -> 0.00 mm
- net Net-(R4-Pad1): track 64.3 -> 0.00 mm
- net Net-(R3-Pad1): track 64.0 -> 0.00 mm
- net Net-(R6-Pad1): track 63.0 -> 0.00 mm, vias 2 -> 0
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
Commit message: update
Parts:
- removed the mountingHole2 at (80.8, 137.7)
- D1: value LED C -> C
- D2: value LED B -> B
- D3: value LED A -> A
- R3, R4, R6: moved to F.Cu
- U15: value WeMos_D1_mini -> WeMos D1 mini
- moved mountingHole1 33.4 mm to (73.0, 136.1)
- moved J1 4.33 mm to (36.1, 147.3)
- moved U18 1.83 mm to (49.5, 131.3), turned to 0 degrees
- moved mountingHole2 1.53 mm to (123.0, 136.1)
- moved R8 1.52 mm to (48.8, 143.3)
- moved U1 1.43 mm to (43.0, 140.7)
- moved U4 1.07 mm to (84.8, 158.1), turned to 0 degrees
- moved C2 1.02 mm to (128.3, 135.4)
- moved U7 1.02 mm to (117.1, 157.5), turned to 0 degrees
- moved U5 0.92 mm to (95.5, 158.0), turned to 0 degrees
- moved JP1 0.76 mm to (78.7, 127.3)
- moved JP2 0.76 mm to (93.0, 127.3)
- moved JP3 0.76 mm to (105.7, 127.3)
- moved JP4 0.76 mm to (118.4, 127.3)
- moved U6 0.51 mm to (105.7, 158.0), turned to 0 degrees
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- renumbered mountingHole3 to mountingHole2
Other:
- board size 100 x 49.3 mm -> 100 x 50 mm
- board text added: "+"
- board text added: "."
